File: erack-14HP.kicad_pcb (KiCad board)
At the start: 2 copper layers, 68.8 x 100 mm, 0 parts

Commit message: Playing around with some ideas for a 14HP foundation
Parts:
- added REF**: Pin_Header_Straight_1x39_Pitch2.54mm, Pin_Headers:Pin_Header_Straight_1x39_Pitch2.54mm, F.Cu at (117.7, 38.0)
- added REF**: Pin_Header_Straight_1x39_Pitch2.54mm, Pin_Headers:Pin_Header_Straight_1x39_Pitch2.54mm, F.Cu at (183.1, 38.0)
