File: 8HP/base/base-UI-8HP.kicad_pcb (KiCad board)
At the start: 2 copper layers, 69.8 x 100 mm, 2 parts

Commit message: A little restructuring...
Parts:
- removed the REF** at (117.0, 39.8)
- removed the REF** at (183.8, 39.8)
- added REF**: Val**, erack:Headers39Male, B.Cu at (153.3, 39.8)
- added REF**: Val**, erack:Headers39Male, B.Cu at (117.0, 39.8)
Other:
- board size 69.8 x 100 mm -> 39.3 x 100 mm
