File: 8HP/base/base-IO-8HP.sch (KiCad schematic (older format))
At the start: 2 parts

Commit message: Starting with the Teensy integration
Parts:
- J1, J2: renamed from J?; footprint (none) -> krachmacher:PinSocket39
Connections:
- net GND: now reaches J1.1 (GND)
- net GND: now also J1.22 (GND), J1.39 (GND), J2.1 (GND), J2.22 (GND), J2.39 (GND)
- net +12VA: now reaches J1.2 (+12V)
- net +12VA: now also J2.2 (+12V)
- net +5V: now reaches J1.3 (+5V)
- net +5V: now also J2.3 (+5V)
- net -12VA: now reaches J1.5 (-12V)
- net -12VA: now also J2.5 (-12V)
Other:
- moved on the sheet: J1, J2
Changed lines of the file:
@@
 $EndDescr
 $Comp
-L _KRACHMACHER:KRACHMACHER_01x39_Input J?
+L _KRACHMACHER:KRACHMACHER_01x39_Input J1
 U 1 1 5A97234A
-P 850 3300
-F 0 "J?" H 730 5417 50  0000 C CNN
-F 1 "IN" H 730 5326 50  0000 C CNN
-F 2 "" H 650 3300 50  0001 C CNN
-F 3 "~" H 650 3300 50  0001 C CNN
-	1    850  3300
+P 950 3300
+F 0 "J1" H 830 5417 50  0000 C CNN
+F 1 "IN" H 830 5326 50  0000 C CNN
+F 2 "krachmacher:PinSocket39" H 750 3300 50  0001 C CNN
+F 3 "~" H 750 3300 50  0001 C CNN
+	1    950  3300
 	1    0    0    -1
 $EndComp
 $Comp
-L _KRACHMACHER:KRACHMACHER_01x39_Output J?
+L _KRACHMACHER:KRACHMACHER_01x39_Output J2
 U 1 1 5A9724BC
-P 11000 3300
-F 0 "J?" H 11050 5450 50  0000 L CNN
-F 1 "OUT" H 11000 5350 50  0000 L CNN
-F 2 "" H 11100 3300 50  0001 C CNN
-F 3 "~" H 11100 3300 50  0001 C CNN
-	1    11000 3300
+P 10800 3300
+F 0 "J2" H 10850 5450 50  0000 L CNN
+F 1 "OUT" H 10800 5350 50  0000 L CNN
+F 2 "krachmacher:PinSocket39" H 10900 3300 50  0001 C CNN
+F 3 "~" H 10900 3300 50  0001 C CNN
+	1    10800 3300
 	1    0    0    -1
 $EndComp
@@
 F1 "base-IO-power.sch" 59
 $EndSheet
+$Comp
+L power:+12VA #PWR0101
+U 1 1 5AA30982
+P 950 1500
+F 0 "#PWR0101" H 950 1350 50  0001 C CNN
+F 1 "+12VA" V 965 1628 50  0000 L CNN
+F 2 "" H 950 1500 50  0001 C CNN
+F 3 "" H 950 1500 50  0001 C CNN
+	1    950  1500
+	0    1    1    0
+$EndComp
+$Comp
+L power:+5V #PWR0102
+U 1 1 5AA309CF
+P 950 1600
+F 0 "#PWR0102" H 950 1450 50  0001 C CNN
+F 1 "+5V" V 965 1728 50  0000 L CNN
+F 2 "" H 950 1600 50  0001 C CNN
+F 3 "" H 950 1600 50  0001 C CNN
+	1    950  1600
+	0    1    1    0
+$EndComp
+$Comp
+L power:-12VA #PWR0104
+U 1 1 5AA30A7E
+P 950 1800
+F 0 "#PWR0104" H 950 1650 50  0001 C CNN
+F 1 "-12VA" V 965 1928 50  0000 L CNN
+F 2 "" H 950 1800 50  0001 C CNN
+F 3 "" H 950 1800 50  0001 C CNN
+	1    950  1800
+	0    1    1    0
+$EndComp
+$Comp
+L power:GND #PWR0105
+U 1 1 5AA30AD9
+P 950 1400
+F 0 "#PWR0105" H 950 1150 50  0001 C CNN
+F 1 "GND" V 955 1272 50  0000 R CNN
+F 2 "" H 950 1400 50  0001 C CNN
+F 3 "" H 950 1400 50  0001 C CNN
+	1    950  1400
+	0    -1   -1   0
+$EndComp
+$Comp
+L power:+12VA #PWR0108
+U 1 1 5AA30B6F
+P 10700 1500
+F 0 "#PWR0108" H 10700 1350 50  0001 C CNN
+F 1 "+12VA" V 10715 1628 50  0000 L CNN
+F 2 "" H 10700 1500 50  0001 C CNN
+F 3 "" H 10700 1500 50  0001 C CNN
+	1    10700 1500
+	0    -1   -1   0
+$EndComp
+$Comp
+L power:+5V #PWR0109
+U 1 1 5AA30B75
+P 10700 1600
+F 0 "#PWR0109" H 10700 1450 50  0001 C CNN
+F 1 "+5V" V 10715 1728 50  0000 L CNN
+F 2 "" H 10700 1600 50  0001 C CNN
+F 3 "" H 10700 1600 50  0001 C CNN
+	1    10700 1600
+	0    -1   -1   0
+$EndComp
+$Comp
+L power:-12VA #PWR0111
+U 1 1 5AA30B81
+P 10700 1800
+F 0 "#PWR0111" H 10700 1650 50  0001 C CNN
+F 1 "-12VA" V 10715 1928 50  0000 L CNN
+F 2 "" H 10700 1800 50  0001 C CNN
+F 3 "" H 10700 1800 50  0001 C CNN
+	1    10700 1800
+	0    -1   -1   0
+$EndComp
+$Comp
+L power:GND #PWR0112
+U 1 1 5AA30B87
+P 10700 3500
+F 0 "#PWR0112" H 10700 3250 50  0001 C CNN
+F 1 "GND" V 10705 3372 50  0000 R CNN
+F 2 "" H 10700 3500 50  0001 C CNN
+F 3 "" H 10700 3500 50  0001 C CNN
+	1    10700 3500
+	0    1    1    0
+$EndComp
+$Comp
+L power:GND #PWR0113
+U 1 1 5AA30B8D
+P 10700 1400
+F 0 "#PWR0113" H 10700 1150 50  0001 C CNN
+F 1 "GND" V 10705 1272 50  0000 R CNN
+F 2 "" H 10700 1400 50  0001 C CNN
+F 3 "" H 10700 1400 50  0001 C CNN
+	1    10700 1400
+	0    1    1    0
+$EndComp
+$Comp
+L power:GND #PWR0114
+U 1 1 5AA30B93
+P 10700 5200
+F 0 "#PWR0114" H 10700 4950 50  0001 C CNN
+F 1 "GND" V 10705 5072 50  0000 R CNN
+F 2 "" H 10700 5200 50  0001 C CNN
+F 3 "" H 10700 5200 50  0001 C CNN
+	1    10700 5200
+	0    1    1    0
+$EndComp
+$Comp
+L power:GND #PWR0107
+U 1 1 5AA30B05
+P 950 3500
+F 0 "#PWR0107" H 950 3250 50  0001 C CNN
+F 1 "GND" V 955 3372 50  0000 R CNN
+F 2 "" H 950 3500 50  0001 C CNN
+F 3 "" H 950 3500 50  0001 C CNN
+	1    950  3500
+	0    -1   -1   0
+$EndComp
+$Comp
+L power:GND #PWR0106
+U 1 1 5AA30AF6
+P 950 5200
+F 0 "#PWR0106" H 950 4950 50  0001 C CNN
+F 1 "GND" V 955 5072 50  0000 R CNN
+F 2 "" H 950 5200 50  0001 C CNN
+F 3 "" H 950 5200 50  0001 C CNN
+	1    950  5200
+	0    -1   -1   0
+$EndComp
 $EndSCHEMATC
