File: 8HP/base/base-IO-power.sch (KiCad schematic (older format))
At the start: 7 parts

Commit message: Progress on the power supply
Parts:
- added C? (x2): CP1, symbol Device:CP1
- added C?: C, Capacitors_SMD:C_0603, symbol Device:C
- added JP?: Jumper_3_Bridged12, Pin_Headers:Pin_Header_Straight_1x03_Pitch2.54mm, symbol Jumper:Jumper_3_Bridged12
- added L? (x4): Ferrite_Bead, Inductors_SMD:L_0603, symbol Device:Ferrite_Bead
- added R?: R, Resistors_SMD:R_0603, symbol Device:R
- added U?: LM1117-3.3, TO_SOT_Packages_SMD:SOT-223, symbol Regulator_Linear:LM1117-3.3
- D? (x3): footprint Diode_THT:D_DO-41_SOD81_Horizontal_RM10 -> Diodes_SMD:D_SOD-123
- J?: footprint (none) -> Pin_Headers:Pin_Header_Straight_2x06_Pitch2.54mm
Connections:
- net labels added: +12VA, +3.3V, +3.3VA
- net labels removed: +12V
- wire segments 36 -> 59
Other:
- moved on the sheet: C?, D?, J?

Commit message: Starting with the Teensy integration
Parts:
- removed C? (x2): CP1, symbol Device:CP1
- removed C?: C, Capacitors_SMD:C_0603, symbol Device:C
- removed JP?: Jumper_3_Bridged12, Pin_Headers:Pin_Header_Straight_1x03_Pitch2.54mm, symbol Jumper:Jumper_3_Bridged12
- removed L?: Ferrite_Bead, Inductors_SMD:L_0603, symbol Device:Ferrite_Bead
- removed R?: R, Resistors_SMD:R_0603, symbol Device:R
- removed U?: LM1117-3.3, TO_SOT_Packages_SMD:SOT-223, symbol Regulator_Linear:LM1117-3.3
- C1: renamed from C?; footprint Capacitors_SMD:CP_Elec_6.3x5.8 -> Capacitors_SMD:CP_Elec_4x5.8
- C2, C3: renamed from C?; footprint (none) -> Capacitors_SMD:CP_Elec_4x5.8
- gave numbers to parts that had none: 7
Connections:
- net labels removed: +3.3V, +3.3VA
- wire segments 59 -> 33
Other:
- moved on the sheet: J3
