File: 8HP/base/base-IO-8HP-teensy.sch (KiCad schematic (older format))
At the start: 13 parts, among them J1 IN, J2 OUT, J3 EURO_POWER_2x6, U1 Teensy3.6

Commit message: Add a simplified Teensy 3.6 symbol and footprint
Parts:
- removed U1: Teensy3.6, krachmacher:Teensy35_36, symbol _KRACHMACHER:Teensy3.6
- added U1: Teensy3.6_Lite, krachmacher:Teensy35_36_Lite, symbol _KRACHMACHER:Teensy3.6_Lite
Connections:
- net +5V: now also U1.53 (Vin)
- net GND: now also U1.1 (GND), U1.39 (GND), U1.52 (AGND)
- net +3V3: now reaches J1.4 (+3.3V)
- net +3V3: now also J2.4 (+3.3V), U1.15 (3.3V), U1.51 (3.3V_max250mA)
Changed lines of the file:
@@
 	2000 6750 2100 6750
 $Comp
-L _KRACHMACHER:Teensy3.6 U1
-U 1 1 5AA9ABE6
-P 5650 2900
-F 0 "U1" H 5650 5287 60  0000 C CNN
-F 1 "Teensy3.6" H 5650 5181 60  0000 C CNN
-F 2 "krachmacher:Teensy35_36" H 5650 2900 60  0000 C CNN
-F 3 "" H 5650 2900 60  0000 C CNN
-	1    5650 2900
+L power:+5V #PWR0121
+U 1 1 5AA9ACF3
+P 6750 850
+F 0 "#PWR0121" H 6750 700 50  0001 C CNN
+F 1 "+5V" V 6765 978 50  0000 L CNN
+F 2 "" H 6750 850 50  0001 C CNN
+F 3 "" H 6750 850 50  0001 C CNN
+	1    6750 850
+	0    1    1    0
+$EndComp
+$Comp
+L power:GND #PWR0122
+U 1 1 5AAADCFF
+P 4550 850
+F 0 "#PWR0122" H 4550 600 50  0001 C CNN
+F 1 "GND" V 4555 722 50  0000 R CNN
+F 2 "" H 4550 850 50  0001 C CNN
+F 3 "" H 4550 850 50  0001 C CNN
+	1    4550 850
+	0    1    1    0
+$EndComp
+$Comp
+L power:GND #PWR0123
+U 1 1 5AAADD6F
+P 6750 950
+F 0 "#PWR0123" H 6750 700 50  0001 C CNN
+F 1 "GND" V 6755 822 50  0000 R CNN
+F 2 "" H 6750 950 50  0001 C CNN
+F 3 "" H 6750 950 50  0001 C CNN
+	1    6750 950
+	0    -1   -1   0
+$EndComp
+$Comp
+L power:+3.3V #PWR0124
+U 1 1 5AAADE13
+P 6750 1050
+F 0 "#PWR0124" H 6750 900 50  0001 C CNN
+F 1 "+3.3V" V 6765 1178 50  0000 L CNN
+F 2 "" H 6750 1050 50  0001 C CNN
+F 3 "" H 6750 1050 50  0001 C CNN
+	1    6750 1050
+	0    1    1    0
+$EndComp
+$Comp
+L power:+3.3V #PWR0125
+U 1 1 5AAADE4C
+P 950 1700
+F 0 "#PWR0125" H 950 1550 50  0001 C CNN
+F 1 "+3.3V" V 965 1828 50  0000 L CNN
+F 2 "" H 950 1700 50  0001 C CNN
+F 3 "" H 950 1700 50  0001 C CNN
+	1    950  1700
+	0    1    1    0
+$EndComp
+$Comp
+L power:+3.3V #PWR0126
+U 1 1 5AAADE71
+P 10700 1700
+F 0 "#PWR0126" H 10700 1550 50  0001 C CNN
+F 1 "+3.3V" V 10715 1828 50  0000 L CNN
+F 2 "" H 10700 1700 50  0001 C CNN
+F 3 "" H 10700 1700 50  0001 C CNN
+	1    10700 1700
+	0    -1   -1   0
+$EndComp
+$Comp
+L power:GND #PWR0127
+U 1 1 5AAADEE1
+P 6750 2250
+F 0 "#PWR0127" H 6750 2000 50  0001 C CNN
+F 1 "GND" V 6755 2122 50  0000 R CNN
+F 2 "" H 6750 2250 50  0001 C CNN
+F 3 "" H 6750 2250 50  0001 C CNN
+	1    6750 2250
+	0    -1   -1   0
+$EndComp
+$Comp
+L _KRACHMACHER:Teensy3.6_Lite U1
+U 1 1 5AAAEB07
+P 5650 2050
+F 0 "U1" H 5650 3643 60  0000 C CNN
+F 1 "Teensy3.6_Lite" H 5650 3537 60  0000 C CNN
+F 2 "krachmacher:Teensy35_36_Lite" H 5650 3431 60  0000 C CNN
+F 3 "" H 5550 1150 60  0000 C CNN
+	1    5650 2050
 	1    0    0    -1
 $EndComp
 $Comp
-L power:+5V #PWR0121
-U 1 1 5AA9ACF3
-P 6650 4100
-F 0 "#PWR0121" H 6650 3950 50  0001 C CNN
-F 1 "+5V" V 6665 4228 50  0000 L CNN
-F 2 "" H 6650 4100 50  0001 C CNN
-F 3 "" H 6650 4100 50  0001 C CNN
-	1    6650 4100
-	0    1    1    0
+L power:+3.3V #PWR0128
+U 1 1 5AAB01E6
+P 4550 2250
+F 0 "#PWR0128" H 4550 2100 50  0001 C CNN
+F 1 "+3.3V" V 4565 2378 50  0000 L CNN
+F 2 "" H 4550 2250 50  0001 C CNN
+F 3 "" H 4550 2250 50  0001 C CNN
+	1    4550 2250
+	0    -1   -1   0
 $EndComp
 $EndSCHEMATC
